File: UINIO-Power-LDO.kicad_pcb (KiCad board)
At the start: 2 copper layers, 0 parts

Commit message: Initialization project.
Parts:
- added C1: 1uF, Capacitor_SMD:C_0603_1608Metric, F.Cu at (149.7, 87.5)
- added C2: 1uF, Capacitor_SMD:C_0603_1608Metric, F.Cu at (149.1, 113.5)
- added C3: 1uF, Capacitor_SMD:C_0603_1608Metric, F.Cu at (149.7, 95.5)
- added C4: 1uF, Capacitor_SMD:C_0603_1608Metric, F.Cu at (149.1, 121.6)
- added C5: 1uF, Capacitor_SMD:C_0603_1608Metric, F.Cu at (150.8, 61.8)
- added C6: 0.01uF, Capacitor_SMD:C_0603_1608Metric, F.Cu at (150.8, 69.0)
- added C7: 1uF, Capacitor_SMD:C_0603_1608Metric, F.Cu at (156.1, 67.6)
- added C8: 10uF, Capacitor_SMD:C_0603_1608Metric, F.Cu at (148.8, 149.3)
- added C9: 22uF, Capacitor_Tantalum_SMD:CP_EIA-3528-15_AVX-H_Pad1.50x2.35mm_HandSolder, F.Cu at (148.7, 138.8)
- added D1: 1N5819, Diode_SMD:Nexperia_CFP3_SOD-123W, F.Cu at (143.6, 91.5)
- added D2: 1N5819, Diode_SMD:Nexperia_CFP3_SOD-123W, F.Cu at (143.6, 117.6)
- added D3: LED_Red, LED_SMD:LED_0603_1608Metric, F.Cu at (155.7, 92.5)
- added D4: 1N5819, Diode_SMD:Nexperia_CFP3_SOD-123W, F.Cu at (140.7, 65.4)
- added D5: LED_Red, LED_SMD:LED_0603_1608Metric, F.Cu at (156.1, 64.8)
- added D6: 1N5819, Diode_SMD:Nexperia_CFP3_SOD-123W, F.Cu at (141.9, 143.7)
- added D7: LED_Red, LED_SMD:LED_0603_1608Metric, F.Cu at (155.1, 118.7)
- added D8: LED_Red, LED_SMD:LED_0603_1608Metric, F.Cu at (156.0, 145.0)
- added HOLE**: Hole-2mm, Uinio:Hole-2mm, F.Cu at (126.6, 57.2)
- added HOLE**: Hole-2mm, Uinio:Hole-2mm, F.Cu at (126.5, 125.8)
- added HOLE**: Hole-2mm, Uinio:Hole-2mm, F.Cu at (126.5, 151.9)
- added HOLE**: Hole-2mm, Uinio:Hole-2mm, F.Cu at (162.8, 73.5)
- added HOLE**: Hole-2mm, Uinio:Hole-2mm, F.Cu at (126.6, 135.6)
- added HOLE**: Hole-2mm, Uinio:Hole-2mm, F.Cu at (126.6, 109.5)
- added HOLE**: Hole-2mm, Uinio:Hole-2mm, F.Cu at (126.5, 73.5)
- added HOLE**: Hole-2mm, Uinio:Hole-2mm, F.Cu at (162.8, 151.9)
- added HOLE**: Hole-2mm, Uinio:Hole-2mm, F.Cu at (162.8, 109.5)
- added HOLE**: Hole-2mm, Uinio:Hole-2mm, F.Cu at (126.5, 99.6)
- added HOLE**: Hole-2mm, Uinio:Hole-2mm, F.Cu at (162.8, 83.3)
- added HOLE**: Hole-2mm, Uinio:Hole-2mm, F.Cu at (162.8, 135.6)
- added HOLE**: Hole-2mm, Uinio:Hole-2mm, F.Cu at (126.6, 83.3)
- added HOLE**: Hole-2mm, Uinio:Hole-2mm, F.Cu at (162.8, 125.7)
- added HOLE**: Hole-2mm, Uinio:Hole-2mm, F.Cu at (162.8, 99.6)
- added HOLE**: Hole-2mm, Uinio:Hole-2mm, F.Cu at (162.8, 57.2)
- added J1: Conn_01x02_Pin, Connector_PinHeader_2.54mm:PinHeader_1x02_P2.54mm_Vertical, F.Cu at (137.5, 90.2)
- added J2: Conn_01x02_Pin, Connector_PinHeader_2.54mm:PinHeader_1x02_P2.54mm_Vertical, F.Cu at (137.4, 116.3)
- added J3: Conn_01x02_Pin, Connector_PinHeader_2.54mm:PinHeader_1x02_P2.54mm_Vertical, F.Cu at (136.0, 64.1)
- added J4: Conn_01x03_Pin, Connector_PinHeader_2.54mm:PinHeader_1x03_P2.54mm_Vertical, F.Cu at (145.4, 62.9)
- added J5: Conn_01x04_Pin, Connector_PinHeader_2.54mm:PinHeader_1x04_P2.54mm_Vertical, F.Cu at (163.3, 61.6)
- added J6: Conn_01x02_Pin, Connector_PinHeader_2.54mm:PinHeader_1x02_P2.54mm_Vertical, F.Cu at (136.3, 142.4)
- added J7: Conn_01x04_Pin, Connector_PinHeader_2.54mm:PinHeader_1x04_P2.54mm_Vertical, F.Cu at (163.3, 87.7)
- added J8: Conn_01x04_Pin, Connector_PinHeader_2.54mm:PinHeader_1x04_P2.54mm_Vertical, F.Cu at (163.3, 139.9)
- added J9: Conn_01x04_Pin, Connector_PinHeader_2.54mm:PinHeader_1x04_P2.54mm_Vertical, F.Cu at (163.3, 113.8)
- added R1: 5.1k, Resistor_SMD:R_0603_1608Metric, F.Cu at (137.4, 86.2)
- added R10: 2K, Resistor_SMD:R_0603_1608Metric, F.Cu at (156.1, 63.2)
- added R11: 2K, Resistor_SMD:R_0603_1608Metric, F.Cu at (155.1, 116.6)
- added R12: 2K, Resistor_SMD:R_0603_1608Metric, F.Cu at (156.0, 142.7)
- added R2: 5.1k, Resistor_SMD:R_0603_1608Metric, F.Cu at (137.5, 96.8)
- added R3: 5.1k, Resistor_SMD:R_0603_1608Metric, F.Cu at (137.4, 112.3)
- added R4: 5.1k, Resistor_SMD:R_0603_1608Metric, F.Cu at (137.4, 122.9)
- added R5: 5.1k, Resistor_SMD:R_0603_1608Metric, F.Cu at (136.0, 60.2)
- added R6: 5.1k, Resistor_SMD:R_0603_1608Metric, F.Cu at (136.0, 70.6)
- added R7: 2K, Resistor_SMD:R_0603_1608Metric, F.Cu at (155.7, 90.3)
- added R8: 5.1k, Resistor_SMD:R_0603_1608Metric, F.Cu at (136.3, 138.4)
- added R9: 5.1k, Resistor_SMD:R_0603_1608Metric, F.Cu at (136.3, 149.0)
- added TP1: TestPoint, TestPoint:TestPoint_Pad_D1.5mm, F.Cu at (143.6, 96.8)
- added TP10: TestPoint, TestPoint:TestPoint_Pad_D1.5mm, F.Cu at (156.1, 70.6)
- added TP11: TestPoint, TestPoint:TestPoint_Pad_D1.5mm, F.Cu at (141.9, 149.0)
- added TP12: TestPoint, TestPoint:TestPoint_Pad_D1.5mm, F.Cu at (156.0, 149.0)
- added TP13: TestPoint, TestPoint:TestPoint_Pad_D1.5mm, F.Cu at (156.1, 60.2)
- added TP14: TestPoint, TestPoint:TestPoint_Pad_D1.5mm, F.Cu at (155.7, 86.2)
- added TP15: TestPoint, TestPoint:TestPoint_Pad_D1.5mm, F.Cu at (156.0, 138.4)
- added TP16: TestPoint, TestPoint:TestPoint_Pad_D1.5mm, F.Cu at (155.1, 122.9)
- added TP2: TestPoint, TestPoint:TestPoint_Pad_D1.5mm, F.Cu at (143.6, 86.2)
- added TP3: TestPoint, TestPoint:TestPoint_Pad_D1.5mm, F.Cu at (143.5, 112.3)
- added TP4: TestPoint, TestPoint:TestPoint_Pad_D1.5mm, F.Cu at (143.6, 122.9)
- added TP5: TestPoint, TestPoint:TestPoint_Pad_D1.5mm, F.Cu at (155.8, 96.8)
- added TP6: TestPoint, TestPoint:TestPoint_Pad_D1.5mm, F.Cu at (140.7, 60.2)
- added TP7: TestPoint, TestPoint:TestPoint_Pad_D1.5mm, F.Cu at (155.1, 112.3)
- added TP8: TestPoint, TestPoint:TestPoint_Pad_D1.5mm, F.Cu at (140.7, 70.6)
- added TP9: TestPoint, TestPoint:TestPoint_Pad_D1.5mm, F.Cu at (141.9, 138.4)
- added U1: ME6211C33M5G-N, Uinio:SOT-23-5_L3.0-W1.7-P0.95-LS2.8-BR, F.Cu at (149.6, 91.5)
- added U2: XC6206PxxxMR, Package_TO_SOT_SMD:SOT-23-3, F.Cu at (149.5, 117.6)
- added U3: SGM2019-3.3YN5G, Uinio:SOT-23-5_L3.0-W1.7-P0.95-LS2.8-BR, F.Cu at (150.6, 65.4)
- added U4: AMS1117, Uinio:SOT-223-3_L6.6-W3.5-P2.30-LS7.0-BL, F.Cu at (148.8, 144.7)
- added USB1: USB_Type_C_6Pin, Uinio:USB-TYPEC-250-BRP6L68, F.Cu at (129.2, 91.5)
- added USB2: USB_Type_C_6Pin, Uinio:USB-TYPEC-250-BRP6L68, F.Cu at (129.2, 117.6)
- added USB3: USB_Type_C_6Pin, Uinio:USB-TYPEC-250-BRP6L68, F.Cu at (129.2, 65.4)
- added USB4: USB_Type_C_6Pin, Uinio:USB-TYPEC-250-BRP6L68, F.Cu at (129.2, 143.7)
Other:
- board outline added: 40 x 98.3 mm
- board text added: "+"
- board text added: "-"
- board text added: "GND"
- board text added: "SOT-223-3"
- board text added: "SOT-23-3"
- board text added: "SOT-23-5"
- board text added: "UINIO-Power-LDO-AMS1117"
- board text added: "UINIO-Power-LDO-ME6211"
- board text added: "UINIO-Power-LDO-SGM2019"
- board text added: "UINIO-Power-LDO-XC6206"
- board text added: "UinIO.com"
- board text added: "VCC"

Commit message: Initialization project.
Routing:
- added copper zone on B.Cu, net GND-SGM2019
- added copper zone on F.Cu, net GND-SGM2019
- added copper zone on B.Cu, net Output-SGM2019
- added copper zone on F.Cu, net Output-SGM2019
Changed lines of the file:
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@@
+		)
+	)
+	(zone
+		(net 4)
+		(net_name "GND-SGM2019")
+		(layers "F&B.Cu")
+		(hatch edge 0.5)
+		(connect_pads yes
+			(clearance 0.5)
+		)
+		(min_thickness 0.25)
+		(filled_areas_thickness no)
+		(fill yes
+			(thermal_gap 0.5)
+			(thermal_bridge_width 0.5)
+		)
+		(polygon
+			(pts
+				(xy 168.94 50.77) (xy 168.94 75.17) (xy 167.23 76.88) (xy 122.44 76.88) (xy 119.82 74.26) (xy 119.82 50.77)
+			)
+		)
+	)
+	(zone
+		(net 28)
+		(net_name "Output-SGM2019")
+		(layers "F&B.Cu")
+		(hatch edge 0.5)
+		(connect_pads yes
+			(clearance 0.5)
+		)
+		(min_thickness 0.25)
+		(filled_areas_thickness no)
+		(fill yes
+			(thermal_gap 0.5)
+			(thermal_bridge_width 0.5)
+		)
+		(polygon
+			(pts
+				(xy 169.02 50.71) (xy 169.02 75.11) (xy 167.31 76.82) (xy 122.52 76.82) (xy 119.9 74.2) (xy 119.9 50.71)
+			)
 		)
 	)
