File: UINIO-Power-LDO.kicad_pcb (KiCad board)
At the start: 2 copper layers, 40 x 98.3 mm, 78 parts, among them J1 Conn_01x02_Pin, J2 Conn_01x02_Pin, J3 Conn_01x02_Pin, J4 Conn_01x03_Pin, J5 Conn_01x04_Pin, J6 Conn_01x02_Pin, J7 Conn_01x04_Pin, J8 Conn_01x04_Pin, J9 Conn_01x04_Pin, U1 ME6211C33M5G-N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

Commit message: Finish PCB Layout.
Parts:
- added HOLE**: Hole-2mm, Uinio:Hole-2mm, F.Cu at (242.4, 161.3)
- added HOLE**: Hole-2mm, Uinio:Hole-2mm, F.Cu at (242.5, 145.1)
- added HOLE**: Hole-2mm, Uinio:Hole-2mm, F.Cu at (278.7, 145.1)
- added HOLE**: Hole-2mm, Uinio:Hole-2mm, F.Cu at (278.7, 161.3)
- moved TP9 10.7 mm to (141.5, 149.1), turned to 180 degrees
- moved TP3 10.7 mm to (143.3, 123.0), turned to 180 degrees
- moved TP7 10.7 mm to (155.1, 123.0)
- moved TP4 10.5 mm to (143.3, 112.4), turned to 180 degrees
- moved TP16 10.5 mm to (155.1, 112.4)
- moved TP11 10.5 mm to (141.5, 138.5), turned to 180 degrees
- moved TP6 10.4 mm to (140.7, 70.6), turned to -90 degrees
- moved TP8 10.3 mm to (140.7, 60.3), turned to -90 degrees
- moved J6 2.55 mm to (136.3, 145.0), turned to 180 degrees
- moved J1 2.55 mm to (137.5, 92.8), turned to 180 degrees
- moved J2 2.55 mm to (137.4, 118.9), turned to 180 degrees
- moved J3 2.55 mm to (136.0, 66.7), turned to 180 degrees
- moved C6 1.06 mm to (149.7, 69.0), turned to 90 degrees
- moved C4 0.90 mm to (149.4, 120.7)
- moved C5 0.84 mm to (151.6, 61.7), turned to -90 degrees
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Connections:
- net Output-AMS1117 renamed VCC-AMS1117
- net Output-ME6211 renamed VCC-ME6211
- net Output-SGM2019 renamed VCC-SGM2019
- net Output-XC6206 renamed VCC-XC6206
- J2 pad 2: GND-ME6211 -> GND-XC6206
- J6 pad 2: GND-SGM2019 -> GND-AMS1117
Routing:
- net VCC-AMS1117: track 0.00 -> 45.7 mm
- net VCC-XC6206: track 0.00 -> 31.1 mm
- net VCC-SGM2019: track 0.00 -> 30.6 mm
- net VCC-ME6211: track 0.00 -> 30.2 mm
- net Net-(D1-A): track 0.00 -> 22.5 mm
- net Net-(D2-A): track 0.00 -> 22.1 mm
- net Net-(D4-K): track 0.00 -> 19.9 mm
- net Net-(D6-A): track 0.00 -> 19.2 mm
- net Net-(D4-A): track 0.00 -> 18.0 mm
- net Net-(D1-K): track 0.00 -> 16.1 mm
- net Net-(D6-K): track 0.00 -> 15.0 mm
- net Net-(D2-K): track 0.00 -> 11.6 mm
- net Net-(USB1-CC2): track 0.00 -> 9.87 mm, vias 0 -> 2
- net Net-(USB2-CC1): track 0.00 -> 9.78 mm, vias 0 -> 2
- net Net-(USB1-CC1): track 0.00 -> 9.77 mm, vias 0 -> 2
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- added copper zone on B.Cu, net GND-AMS1117
- added copper zone on F.Cu, net GND-AMS1117
- added copper zone on B.Cu, net GND-ME6211
- added copper zone on F.Cu, net GND-ME6211
- added copper zone on B.Cu, net GND-XC6206
- added copper zone on F.Cu, net GND-XC6206
- removed copper zone on B.Cu, net VCC-SGM2019
- removed copper zone on F.Cu, net VCC-SGM2019

Commit message: Finish PCB Layout.
Parts:
- removed the HOLE** at (242.4, 161.3)
- removed the HOLE** at (242.5, 145.1)
- removed the HOLE** at (278.7, 145.1)
- removed the HOLE** at (278.7, 161.3)
- added HOLE**: Hole-2.6mm, Uinio:Hole-2.6mm, F.Cu at (145.2, 104.5)
- added HOLE**: Hole-2.6mm, Uinio:Hole-2.6mm, F.Cu at (145.2, 78.5)
- added HOLE**: Hole-2.6mm, Uinio:Hole-2.6mm, F.Cu at (145.2, 130.6)
Routing:
- net VCC-AMS1117: track 45.7 -> 39.7 mm
Other:
- outline, holes or cut-outs redrawn
- board text added: "Version 1.0.0"
