File: UINIO-Power-LDO.kicad_pcb (KiCad board)
At the start: 2 copper layers, 40 x 98.3 mm, 81 parts, among them J1 Conn_01x02_Pin, J2 Conn_01x02_Pin, J3 Conn_01x02_Pin, J4 Conn_01x03_Pin, J5 Conn_01x04_Pin, J6 Conn_01x02_Pin, J7 Conn_01x04_Pin, J8 Conn_01x04_Pin, J9 Conn_01x04_Pin, U1 ME6211C33M5G-N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

Commit message: Releaase UINIO-Power-LDO version 2.0.0.
Other:
- board text added: "Version 2.0.0"
- board text removed: "Version 1.0.0"
