File: UINIO-Power-LDO.kicad_sch (KiCad schematic)
At the start: 0 parts

Commit message: Initialization project.
Parts:
- added C1, C2, C3: 1uF, Capacitor_SMD:C_0402_1005Metric, symbol Device:C
- added C4, C5: 1uF, Capacitor_SMD:C_0603_1608Metric, symbol Device:C
- added C6: 0.01uF, Capacitor_SMD:C_0603_1608Metric, symbol Device:C
- added C7, C8: 10uF, Capacitor_SMD:C_0402_1005Metric, symbol Device:C
- added D1, D4: LED_Red, LED_SMD:LED_0603_1608Metric, symbol Device:LED
- added D2: 1N5819, Diode_SMD:D_SOD-323F, symbol Diode:1N5819
- added D3: 1N5819, Diode_SMD:D_SOD-123, symbol Diode:1N5819
- added J1: Conn_01x03_Pin, symbol Connector:Conn_01x03_Pin
- added R1: 2K, Resistor_SMD:R_0402_1005Metric, symbol Device:R
- added R2: 512R, Resistor_SMD:R_0603_1608Metric, symbol Device:R
- added R3: 2K, Resistor_SMD:R_0603_1608Metric, symbol Device:R
- added U1: ME6211C33M5G-N, Uinio:SOT-23-5_L3.0-W1.7-P0.95-LS2.8-BR, symbol Uinio:ME6211
- added U2: XC6206PxxxMR, Package_TO_SOT_SMD:SOT-23-3, symbol Regulator_Linear:XC6206PxxxMR
- added U3: SGM2019-3.3YN5G, Uinio:SOT-23-5_L3.0-W1.7-P0.95-LS2.8-BR, symbol Uinio:SGM2019-3.3YN5G
- added U4: AMS1117, Uinio:SOT-223-3_L6.6-W3.5-P2.30-LS7.0-BL, symbol Uinio:AMS1117
- added USB1, USB2, USB3, USB4: USB_Type_C_6Pin, Uinio:USB-TYPEC-250-BRP6L68, symbol Uinio:USB_Type_C_6Pin
Connections:
- new net: D2.2 (A), USB2.A9 (VBUS), USB2.B9 (VBUS)
- new net: C1.2, U1.1 (Vin), U1.3 (CE), USB1.A9 (VBUS), USB1.B9 (VBUS)
- new net: D1.2 (A), R1.1
- new net: C4.2, D3.1 (K), R2.1, U3.1 (IN)
- new net: C6.2, U3.4 (FB)
- new net: D3.2 (A), USB4.A9 (VBUS), USB4.B9 (VBUS)
- new net: C7.1, U4.3 (Vin), USB3.A9 (VBUS), USB3.B9 (VBUS)
- new net: D4.2 (A), R3.1
- new net: D2.1 (K), U2.3 (VI)
- new net 3.3V_0.96_OLED: C3.1, U2.2 (VO)
- new net GND: C1.1, C2.1, C3.2, C4.1, C5.1, C6.1, C7.2, C8.2, D1.1 (K), D4.1 (K), U1.2 (Vss), U2.1 (GND), U3.2 (GND), U4.1 (GND), USB1.1 (GND), USB1.2 (GND), USB1.3 (GND), USB1.4 (GND), USB1.A12 (GND), USB1.B12 (GND), USB2.1 (GND), USB2.2 (GND), USB2.3 (GND), USB2.4 (GND), USB2.A12 (GND), USB2.B12 (GND), USB3.1 (GND), USB3.2 (GND), USB3.3 (GND), USB3.4 (GND), USB3.A12 (GND), USB3.B12 (GND), USB4.1 (GND), USB4.2 (GND), USB4.3 (GND), USB4.4 (GND), USB4.A12 (GND), USB4.B12 (GND)
- new net LDO_EN: R2.2, U3.3 (EN)
- new net VDD_3.3V: C2.2, C5.2, C8.1, R1.2, R3.2, U1.5 (Vout), U3.5 (OUT), U4.2 (Vout), U4.4 (Vout)
- no-connect marks 0 -> 9

Commit message: Initialization project.
Parts:
- D2: footprint Diode_SMD:D_SOD-323F -> Diode_THT:D_DO-41_SOD81_P10.16mm_Horizontal
- D3: footprint Diode_SMD:D_SOD-123 -> Diode_THT:D_DO-41_SOD81_P10.16mm_Horizontal
- U4: footprint Uinio:SOT-223-3_L6.6-W3.5-P2.30-LS7.0-BL -> kicad_lceda:SOT-223-3_L6.6-W3.5-P2.30-LS7.0-BL
Connections:
- net LDO_EN is gone; now on an unnamed net: R2.2, U3.3 (EN)
- net GND: now also J1.1 (Pin_1)
- net VDD_3.3V: now also J1.3 (Pin_3)
Other:
- moved on the sheet: C4, C5, C6, C7, D3, D4, J1, R2, R3, U3, USB4

Commit message: Initialization project.
Parts:
- added D5, D6: 1N5819, Diode_THT:D_DO-41_SOD81_P10.16mm_Horizontal, symbol Diode:1N5819
- added J2, J3, J4, J5: Conn_01x02_Pin, Connector_PinHeader_2.54mm:PinHeader_1x02_P2.54mm_Vertical, symbol Connector:Conn_01x02_Pin
- added R10, R11, R4, R5, R6, R7, R8, R9: 5.1k, Resistor_SMD:R_0603_1608Metric, symbol Device:R
- added TP1, TP2, TP3, TP4, TP5, TP6, TP7, TP8: TestPoint, TestPoint:TestPoint_Pad_1.5x1.5mm, symbol Connector:TestPoint
- C1, C2, C3, C7, C8: footprint Capacitor_SMD:C_0402_1005Metric -> Capacitor_SMD:C_0603_1608Metric
- J1: footprint (none) -> Connector_PinHeader_2.54mm:PinHeader_1x03_P2.54mm_Vertical
- R1: footprint Resistor_SMD:R_0402_1005Metric -> Resistor_SMD:R_0603_1608Metric
- U4: footprint kicad_lceda:SOT-223-3_L6.6-W3.5-P2.30-LS7.0-BL -> Uinio:SOT-223-3_L6.6-W3.5-P2.30-LS7.0-BL
Connections:
- net at USB2.A5 (CC1): now also R7.1
- net at D2.2 (A), USB2.A9 (VBUS), USB2.B9 (VBUS): now also J5.1 (Pin_1), TP2.1
- net at USB2.B5 (CC2): now also R6.1
- net at USB1.A5 (CC1): now also R9.1
- net at C1.2, U1.1 (Vin), U1.3 (CE): now also D6.1 (K), TP8.1; no longer USB1.A9 (VBUS), USB1.B9 (VBUS)
- net at USB1.B5 (CC2): now also R8.1
- net at C4.2, D3.1 (K), R2.1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: now also J1.3 (Pin_3), TP4.1
- net at USB4.A5 (CC1): now also R10.1
- net at D3.2 (A), USB4.A9 (VBUS), USB4.B9 (VBUS): now also J3.1 (Pin_1), TP3.1
- net at USB4.B5 (CC2): now also R11.1
- net at USB3.A9 (VBUS), USB3.B9 (VBUS): now also D5.2 (A), J4.1 (Pin_1), TP6.1; no longer C7.1, U4.3 (Vin)
- net at D2.1 (K), U2.3 (VI): now also TP1.1
- net at USB3.A5 (CC1): now also R4.2
- net at USB3.B5 (CC2): now also R5.1
- net 3.3V_0.96_OLED renamed Output_XC6206
- removed net GND: C1.1, C2.1, C3.2, C4.1, C5.1, C6.1, C7.2, C8.2, D1.1 (K), D4.1 (K), J1.1 (Pin_1), U1.2 (Vss), U2.1 (GND), U3.2 (GND), U4.1 (GND), USB1.1 (GND), USB1.2 (GND), USB1.3 (GND), USB1.4 (GND), USB1.A12 (GND), USB1.B12 (GND), USB2.1 (GND), USB2.2 (GND), USB2.3 (GND), USB2.4 (GND), USB2.A12 (GND), USB2.B12 (GND), USB3.1 (GND), USB3.2 (GND), USB3.3 (GND), USB3.4 (GND), USB3.A12 (GND), USB3.B12 (GND), USB4.1 (GND), USB4.2 (GND), USB4.3 (GND), USB4.4 (GND), USB4.A12 (GND), USB4.B12 (GND)
- removed net VDD_3.3V: C2.2, C5.2, C8.1, J1.3 (Pin_3), R1.2, R3.2, U1.5 (Vout), U3.5 (OUT), U4.2 (Vout), U4.4 (Vout)
- new net: D6.2 (A), J2.1 (Pin_1), TP7.1, USB1.A9 (VBUS), USB1.B9 (VBUS)
- new net: C7.1, D5.1 (K), TP5.1, U4.3 (Vin)
- new net GND-AMS1117: C7.2, C8.2, R4.1, R5.2, U4.1 (GND), USB3.1 (GND), USB3.2 (GND), USB3.3 (GND), USB3.4 (GND), USB3.A12 (GND), USB3.B12 (GND)
- new net GND-ME6211: C1.1, C2.1, D1.1 (K), J2.2 (Pin_2), J5.2 (Pin_2), R8.2, R9.2, U1.2 (Vss), USB1.1 (GND), USB1.2 (GND), USB1.3 (GND), USB1.4 (GND), USB1.A12 (GND), USB1.B12 (GND)
- new net GND-SGM2019: C4.1, C5.1, C6.1, D4.1 (K), J1.1 (Pin_1), J3.2 (Pin_2), J4.2 (Pin_2), R10.2, R11.2, U3.2 (GND), USB4.1 (GND), USB4.2 (GND), USB4.3 (GND), USB4.4 (GND), USB4.A12 (GND), USB4.B12 (GND)
- new net GND-XC6206: C3.2, R6.2, R7.2, U2.1 (GND), USB2.1 (GND), USB2.2 (GND), USB2.3 (GND), USB2.4 (GND), USB2.A12 (GND), USB2.B12 (GND)
- new net Output_AMS1117: C8.1, U4.2 (Vout), U4.4 (Vout)
- new net Output_ME6211: C2.2, R1.2, U1.5 (Vout)
- new net Output_SGM2019: C5.2, R3.2, U3.5 (OUT)
- no-connect marks 9 -> 1
Other:
- note added: "AMS1117 线性稳压器"
- note added: "ME6211 低压差线性稳压器"
- note added: "SGM2019 低压差线性稳压器"
- note added: "XC6206 低压差线性稳压器"
- moved on the sheet: C1, C2, C3, C4, C5, C6, C7, C8, D1, D2, D3, D4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

Commit message: Initialization project.
Parts:
- removed R2: 512R, Resistor_SMD:R_0603_1608Metric, symbol Device:R
- added C2: 1uF, Capacitor_SMD:C_0603_1608Metric, symbol Device:C
- added D7, D8: LED_Red, LED_SMD:LED_0603_1608Metric, symbol Device:LED
- added J5, J7, J8, J9: Conn_01x04_Pin, Connector_PinHeader_2.54mm:PinHeader_1x04_P2.54mm_Vertical, symbol Connector:Conn_01x04_Pin
- added R11, R12: 2K, Resistor_SMD:R_0603_1608Metric, symbol Device:R
- added TP10, TP12, TP13, TP14, TP15, TP16, TP5, TP7: TestPoint, TestPoint:TestPoint_Pad_D1.5mm, symbol Connector:TestPoint
- C9: renamed from C8; value 10uF -> 22uF; footprint Capacitor_SMD:C_0603_1608Metric -> Capacitor_Tantalum_SMD:CP_EIA-3528-15_AVX-H_Pad1.50x2.35mm_HandSolder
- D1: renamed from D6; footprint Diode_THT:D_DO-41_SOD81_P10.16mm_Horizontal -> Diode_SMD:Nexperia_CFP3_SOD-123W
- D2: footprint Diode_THT:D_DO-41_SOD81_P10.16mm_Horizontal -> Diode_SMD:Nexperia_CFP3_SOD-123W
- D4: renamed from D3; footprint Diode_THT:D_DO-41_SOD81_P10.16mm_Horizontal -> Diode_SMD:Nexperia_CFP3_SOD-123W
- D6: renamed from D5; footprint Diode_THT:D_DO-41_SOD81_P10.16mm_Horizontal -> Diode_SMD:Nexperia_CFP3_SOD-123W
- TP1: renamed from TP7; footprint TestPoint:TestPoint_Pad_1.5x1.5mm -> TestPoint:TestPoint_Pad_D1.5mm
- TP11: renamed from TP5; footprint TestPoint:TestPoint_Pad_1.5x1.5mm -> TestPoint:TestPoint_Pad_D1.5mm
- TP2: renamed from TP8; footprint TestPoint:TestPoint_Pad_1.5x1.5mm -> TestPoint:TestPoint_Pad_D1.5mm
- TP3: renamed from TP2; footprint TestPoint:TestPoint_Pad_1.5x1.5mm -> TestPoint:TestPoint_Pad_D1.5mm
- TP4: renamed from TP1; footprint TestPoint:TestPoint_Pad_1.5x1.5mm -> TestPoint:TestPoint_Pad_D1.5mm
- TP6: renamed from TP3; footprint TestPoint:TestPoint_Pad_1.5x1.5mm -> TestPoint:TestPoint_Pad_D1.5mm
- TP8: renamed from TP4; footprint TestPoint:TestPoint_Pad_1.5x1.5mm -> TestPoint:TestPoint_Pad_D1.5mm
- TP9: renamed from TP6; footprint TestPoint:TestPoint_Pad_1.5x1.5mm -> TestPoint:TestPoint_Pad_D1.5mm
- renumbered C2 to C3, C3 to C4, C4 to C5, C5 to C7, C7 to C8, D1 to D3, D4 to D5, J2 to J1, J5 to J2, J1 to J4, J4 to J6, R9 to R1, R3 to R10, R8 to R2, R7 to R3, R6 to R4, R10 to R5, R11 to R6, R1 to R7, R4 to R8, R5 to R9, USB4 to USB3, USB3 to USB4
Connections:
- net GND-AMS1117: now also D8.1 (K), J8.1 (Pin_1), J8.3 (Pin_3), TP15.1
- net GND-ME6211: now also J7.1 (Pin_1), J7.3 (Pin_3), TP14.1
- net GND-SGM2019: now also J5.1 (Pin_1), J5.3 (Pin_3), TP13.1
- net GND-XC6206: now also C2.2, D7.1 (K), J9.1 (Pin_1), J9.3 (Pin_3), TP16.1
- net at D2.1 (K), TP4.1, U2.3 (VI): now also C2.1
- net Output_AMS1117 renamed Output-AMS1117
- net Output-AMS1117: now also J8.2 (Pin_2), J8.4 (Pin_4), R12.1, TP12.1
- net Output_ME6211 renamed Output-ME6211
- net Output-ME6211: now also J7.2 (Pin_2), J7.4 (Pin_4), TP5.1
- net Output_SGM2019 renamed Output-SGM2019
- net Output-SGM2019: now also J5.2 (Pin_2), J5.4 (Pin_4), TP10.1
- net Output_XC6206 renamed Output-XC6206
- net Output-XC6206: now also J9.2 (Pin_2), J9.4 (Pin_4), R11.2, TP7.1
- new net: D7.2 (A), R11.1
- new net: D8.2 (A), R12.2
Other:
- moved on the sheet: C1, C3, C4, C5, C6, C7, C8, C9, D1, D2, D3, D4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

Commit message: Finish PCB Layout.
Connections:
- net GND-AMS1117: now also J6.2 (Pin_2)
- net GND-ME6211: no longer J2.2 (Pin_2)
- net GND-SGM2019: no longer J6.2 (Pin_2)
- net GND-XC6206: now also J2.2 (Pin_2)
- net Output-AMS1117 renamed VCC-AMS1117
- net Output-ME6211 renamed VCC-ME6211
- net Output-SGM2019 renamed VCC-SGM2019
- net Output-XC6206 renamed VCC-XC6206
Changed lines of the file:
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@@
 			)
 		)
-		(property "Value" "Output-XC6206"
-			(at 157.734 162.052 90)
+		(property "Value" "VCC-XC6206"
+			(at 157.48 165.1 90)
 			(effects
 				(font
@@
 			)
 		)
-		(property "Value" "Output-XC6206"
+		(property "Value" "VCC-XC6206"
 			(at 270.764 149.86 90)
 			(effects
@@
 			)
 		)
-		(property "Value" "Output-XC6206"
+		(property "Value" "VCC-XC6206"
 			(at 271.018 144.78 90)
 			(effects
@@
 			)
 		)
-		(property "Value" "Output-AMS1117"
+		(property "Value" "VCC-AMS1117"
 			(at 245.618 144.78 90)
 			(effects
@@
 			)
 		)
-		(property "Value" "GND-SGM2019"
+		(property "Value" "GND-AMS1117"
 			(at 211.582 95.25 90)
 			(effects
@@
 			)
 		)
-		(property "Value" "Output-SGM2019"
+		(property "Value" "VCC-SGM2019"
 			(at 224.79 29.972 90)
 			(effects
@@
 			)
 		)
-		(property "Value" "Output-SGM2019"
+		(property "Value" "VCC-SGM2019"
 			(at 192.024 149.86 90)
 			(effects
@@
 			)
 		)
-		(property "Value" "Output-AMS1117"
+		(property "Value" "VCC-AMS1117"
 			(at 245.364 149.86 90)
 			(effects
@@
 			)
 		)
-		(property "Value" "Output-SGM2019"
+		(property "Value" "VCC-SGM2019"
 			(at 192.278 144.78 90)
 			(effects
@@
 			)
 		)
-		(property "Value" "GND-ME6211"
+		(property "Value" "GND-XC6206"
 			(at 83.312 154.94 90)
 			(effects
@@
 			)
 		)
-		(property "Value" "Output-ME6211"
+		(property "Value" "VCC-ME6211"
 			(at 133.35 87.122 90)
 			(effects
@@
 			)
 		)
-		(property "Value" "Output-ME6211"
+		(property "Value" "VCC-ME6211"
 			(at 218.694 149.86 90)
 			(effects
@@
 			)
 		)
-		(property "Value" "Output-ME6211"
+		(property "Value" "VCC-ME6211"
 			(at 218.948 144.78 90)
 			(effects
@@
 			)
 		)
-		(property "Value" "Output-AMS1117"
+		(property "Value" "VCC-AMS1117"
 			(at 263.906 81.026 90)
 			(effects
